Commit message: first commit

File: description/gz_diff_drive_control.xacro (robot description, xacro)
@@ -8,5 +8,5 @@
             <right_joint>right_wheel_joint</right_joint>
             <wheel_separation>0.266</wheel_separation>
-            <wheel_radius>0.034</wheel_radius>
+            <wheel_radius>0.05</wheel_radius>
             <!-- Limits -->
             <max_wheel_torque>200</max_wheel_torque>

File: description/lidar.xacro (robot description, xacro)
@@ -1,34 +1,51 @@
 <?xml version="1.0"?>
 <robot xmlns:xacro="http://www.ros.org/wiki/xacro" name="robot">
-    <xacro:property name="lidar_radius"             value="0.025"/>
-    <xacro:property name="lidar_thickness"          value="0.040"/>
-    <xacro:property name="lidar_offset_x"           value="0.230"/>
-    <xacro:property name="lidar_offset_z"           value="0.098"/>
+    <xacro:property name="lidar_radius" value="0.025" />
+    <xacro:property name="lidar_thickness" value="0.040" />
+    <xacro:property name="lidar_offset_x" value="0.230" />
+    <xacro:property name="lidar_offset_z" value="0.098" />
     <!-- Lidar -->
-    <joint name="lidar_joint" type="fixed">
-        <parent link="chasis"/>
-        <child link="lidar_frame"/>
-        <origin xyz="${lidar_offset_x} 0.0 ${lidar_offset_z}" rpy="0 0 ${pi}"/>
+    <joint name="laser_joint" type="fixed">
+        <origin xyz="0.029644 0 0.071347" rpy="0 0 0" />
+        <parent link="base_link" />
+        <child link="laser_frame" />
+        <axis xyz="0 0 1" />
     </joint>
-    <link name="lidar_frame">
+    <link name="laser_frame">
+        <inertial>
+            <origin
+                xyz="0 0 0"
+                rpy="0 0 0" />
+            <mass
+                value="0" />
+            <inertia
+                ixx="0"
+                ixy="0"
+                ixz="0"
+                iyy="0"
+                iyz="0"
+                izz="0" />
+        </inertial>
         <visual>
+            <origin xyz="0 0 0" rpy="0 0 0" />
             <geometry>
-                <cylinder radius="${lidar_radius}" length="${lidar_thickness}"/>
+                <mesh filename="file://$(find halfonso)/meshes/laser_frame.STL" />
             </geometry>
-            <material name="orange"/>
+            <material name="">
+                <color
+                    rgba="1 1 1 1" />
+            </material>
         </visual>
         <collision>
+            <origin xyz="0 0 0" rpy="0 0 0" />
             <geometry>
-                <cylinder radius="${lidar_radius}" length="${lidar_thickness}"/>
+                <mesh filename="file://$(find halfonso)/meshes/laser_frame.STL" />
             </geometry>
         </collision>
-        <xacro:inertial_cylinder mass="0.1" radius="${lidar_radius}" length="${lidar_thickness}">
-            <origin xyz="0 0 0" rpy="0 0 0"/>
-        </xacro:inertial_cylinder>
     </link>
     <!-- Lidar in gazebo-->
-    <gazebo reference="lidar_frame">
+    <gazebo reference="laser_frame">
         <sensor name="lidar" type="gpu_lidar">
-            <gz_frame_id>lidar_frame</gz_frame_id>
+            <gz_frame_id>laser_frame</gz_frame_id>
             <pose>0 0 0 0 0 0</pose>
             <topic>scan</topic>
@@ -62,8 +79,8 @@
                 </noise>
             </lidar>
-        <plugin filename="gz-sim-sensors-system"
+            <plugin filename="gz-sim-sensors-system"
                 name="gz::sim::systems::Sensors">
                 <render_engine>ogre2</render_engine>
-        </plugin>
+            </plugin>
         </sensor>
     </gazebo>

File: description/robot.urdf.xacro (robot description, xacro)
@@ -1,18 +1,18 @@
 <?xml version="1.0"?>
-<robot xmlns:xacro="http://www.ros.org/wiki/xacro"  name="robot">
-    <xacro:arg name="use_ros2_control"              default="true"/>
-    <xacro:arg name="use_ros2_control_gz_sim"       default="false"/>
+<robot xmlns:xacro="http://www.ros.org/wiki/xacro" name="robot">
+    <xacro:arg name="use_ros2_control" default="true" />
+    <xacro:arg name="use_ros2_control_gz_sim" default="false" />
     <!-- Robot_frames -->
-    <xacro:include filename = "robot_main.xacro" />
+    <xacro:include filename="robot_core.xacro" />
     <!-- Controls -->
     <xacro:if value="$(arg use_ros2_control)">
-        <xacro:include filename = "ros2_control.xacro" />
+        <xacro:include filename="ros2_control.xacro" />
     </xacro:if>
     <xacro:unless value="$(arg use_ros2_control)">
-        <xacro:include filename = "gz_diff_drive_control.xacro" />
+        <xacro:include filename="gz_diff_drive_control.xacro" />
     </xacro:unless>
     <!-- Sensors -->
-    <xacro:include filename = "lidar.xacro" />
+    <xacro:include filename="lidar.xacro" />
     <!-- <xacro:include filename = "camera.xacro" /> -->
-    <xacro:include filename = "depth_camera.xacro" />
+    <!-- <xacro:include filename = "depth_camera.xacro" /> -->
 </robot>

File: description/ros2_control.xacro (robot description, xacro)
@@ -5,11 +5,11 @@
             <hardware>
                 <plugin>diffdrive_arduino/DiffDriveArduinoHardware</plugin>
-                    <param name="left_wheel_name">left_wheel_joint</param>
-                    <param name="right_wheel_name">right_wheel_joint</param>
-                    <param name="loop_rate">30</param>
-                    <param name="device">/dev/ttyUSB1</param>
-                    <param name="baud_rate">115200</param>
-                    <param name="timeout_ms">1000</param>
-                    <param name="enc_counts_per_rev">616</param>
+                <param name="left_wheel_name">left_wheel_joint</param>
+                <param name="right_wheel_name">right_wheel_joint</param>
+                <param name="loop_rate">30</param>
+                <param name="device">/dev/serial/by-id/usb-FTDI_FT232R_USB_UART_A5069RR4-if00-port0</param>
+                <param name="baud_rate">57600</param>
+                <param name="timeout_ms">1000</param>
+                <param name="enc_counts_per_rev">2683</param>
             </hardware>
             <joint name="left_wheel_joint">
@@ -18,6 +18,6 @@
                     <param name="max">10</param>
                 </command_interface>
-                <state_interface name="position"/>
-                <state_interface name="velocity"/>
+                <state_interface name="position" />
+                <state_interface name="velocity" />
             </joint>
             <joint name="right_wheel_joint">
@@ -26,11 +26,11 @@
                     <param name="max">10</param>
                 </command_interface>
-                <state_interface name="position"/>
-                <state_interface name="velocity"/>
+                <state_interface name="position" />
+                <state_interface name="velocity" />
             </joint>
         </ros2_control>
     </xacro:unless>
     <xacro:if value="$(arg use_ros2_control_gz_sim)">
-        <ros2_control name="minibot_ros2_control" type="system">
+        <ros2_control name="halfonso_ros2_control" type="system">
             <hardware>
                 <plugin>gz_ros2_control/GazeboSimSystem</plugin>
@@ -41,6 +41,6 @@
                     <param name="max">10</param>
                 </command_interface>
-                <state_interface name="velocity"/>
-                <state_interface name="position"/>
+                <state_interface name="velocity" />
+                <state_interface name="position" />
             </joint>
             <joint name="right_wheel_joint">
@@ -49,6 +49,6 @@
                     <param name="max">10</param>
                 </command_interface>
-                <state_interface name="velocity"/>
-                <state_interface name="position"/>
+                <state_interface name="velocity" />
+                <state_interface name="position" />
             </joint>
         </ros2_control>
@@ -57,5 +57,5 @@
                 name="gz_ros2_control::GazeboSimROS2ControlPlugin">
                 <parameters>
-                    $(find minibot)/config/controller_gz_sim.yaml
+                    $(find halfonso)/config/controller_gz_sim.yaml
                 </parameters>
             </plugin>
